File: pcb/pcb.kicad_pcb (KiCad board)
At the start: 2 copper layers, 108.7 x 45.2 mm, 22 parts, among them SW1 SW_Push, U1 ATmega32U4-AU, Y1 Crystal_GND24_Small

Commit message: finished tracing pcb
Parts:
- removed D1, D2, D3: D_Small, Diode_SMD:D_SOD-123
- moved SW1 78.2 mm to (24.7, 37.1)
- moved C7 77.2 mm to (35.9, 17.5)
- moved C6 71.0 mm to (45.6, 17.7), turned to 180 degrees
- moved R1 67.8 mm to (30.8, 33.6), turned to 90 degrees
- moved R4 65.3 mm to (48.5, 21.8), turned to 270 degrees
- moved MX1 65.0 mm to (61.9, 31.0)
- moved MX2 65.0 mm to (81.0, 31.0)
- moved MX3 65.0 mm to (100.0, 31.0)
- moved C1 62.4 mm to (47.7, 38.0), turned to 270 degrees
- moved Y1 62.1 mm to (43.7, 38.1), turned to 180 degrees
- moved C2 61.6 mm to (39.8, 38.1)
- moved U1 59.2 mm to (40.4, 26.7)
- moved USB1 58.9 mm to (16.9, 29.3)
- moved R2 58.9 mm to (26.3, 29.9)
- moved F1 58.7 mm to (27.1, 24.4)
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Connections:
- MX1 pad 2: Net-(D1-Pad2) -> ROW0
- MX2 pad 2: Net-(D2-Pad2) -> ROW0
- MX3 pad 2: Net-(D3-Pad2) -> ROW0
- U1 pad 26: Net-(U1-Pad26) -> ROW0
- U1 pad 27: Net-(U1-Pad27) -> COL2
- U1 pad 28: Net-(U1-Pad28) -> COL1
- U1 pad 29: Net-(U1-Pad29) -> COL0
- USB1 pad 6: Net-(USB1-Pad6) -> GND
Routing:
- net ROW0: track 38.1 -> 105.1 mm
- net COL2: track 0.00 -> 58.0 mm
- net COL1: track 0.00 -> 43.4 mm
- net +5V: track 119.3 -> 89.4 mm, vias 2 -> 4
- net Net-(R3-Pad1): track 32.8 -> 9.99 mm
- net Net-(R2-Pad1): track 32.0 -> 10.7 mm
- net COL0: track 0.00 -> 20.8 mm
- net GND: track 135.6 -> 116.9 mm
- net Net-(C2-Pad1): track 22.4 -> 7.61 mm
- net Net-(R1-Pad2): track 30.0 -> 17.9 mm
- net Net-(D1-Pad2): track 8.20 -> 0.00 mm
- net Net-(D3-Pad2): track 8.18 -> 0.00 mm
- net Net-(D2-Pad2): track 8.18 -> 0.00 mm
- net Net-(R4-Pad2): track 8.31 -> 2.45 mm
- net Net-(C1-Pad2): track 16.4 -> 18.5 mm
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Other:
- board size 108.7 x 45.2 mm -> 100 x 29.4 mm
- board text added: "three.mee42.dev"
- board text added: "v0.1"

Commit message: de v
Other:
- board text added: "v0.1-dev"
- board text removed: "v0.1"
Changed lines of the file:
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@@
     )
   )
-  (gr_text v0.1 (at 19.939 18.923) (layer F.SilkS)
+  (gr_text v0.1-dev (at 21.844 18.923) (layer F.SilkS)
     (effects (font (size 1 1) (thickness 0.15)))
   )

Commit message: atmega v0.1?
Routing:
- net GND: track 116.9 -> 98.6 mm
- added copper zone on F.Cu, net GND
Changed lines of the file:
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@@
     (thickness 1.6)
     (drawings 10)
-    (tracks 187)
+    (tracks 184)
     (zones 0)
     (modules 19)
@@
     (33 F.Adhes user)
     (34 B.Paste user)
-    (35 F.Paste user)
+    (35 F.Paste user hide)
     (36 B.SilkS user)
     (37 F.SilkS user)
@@
     (last_trace_width 0.254)
     (trace_clearance 0.2)
-    (zone_clearance 0.508)
+    (zone_clearance 0.2)
     (zone_45_only no)
     (trace_min 0.2)
@@
     (add_net VCC)
   )
+  (module Crystal:Crystal_SMD_3225-4Pin_3.2x2.5mm (layer F.Cu)
+    (at 43.67675 38.0755 180)
+    (descr "SMD Crystal SERIES SMD3225/4 http://www.txccrystal.com/images/pdf/7m-accuracy.pdf, 3.2x2.5mm^2 package")
+    (tags "SMD SMT crystal")
+    (attr smd)
+    (fp_text reference Y1 (at -0.01125 2.3885 180) (layer F.SilkS)
+      (effects (font (size 1 1) (thickness 0.15)))
+    )
+    (fp_text value Crystal_GND24_Small (at 0 2.45 180) (layer F.Fab)
+      (effects (font (size 1 1) (thickness 0.15)))
+    )
+    (fp_text user %R (at 0 0 180) (layer F.Fab)
+      (effects (font (size 0.7 0.7) (thickness 0.105)))
+    )
+    (fp_line (start -1.6 -1.25) (end -1.6 1.25) (layer F.Fab) (width 0.1))
+    (fp_line (start -1.6 1.25) (end 1.6 1.25) (layer F.Fab) (width 0.1))
+    (fp_line (start 1.6 1.25) (end 1.6 -1.25) (layer F.Fab) (width 0.1))
+    (fp_line (start 1.6 -1.25) (end -1.6 -1.25) (layer F.Fab) (width 0.1))
+    (fp_line (start -1.6 0.25) (end -0.6 1.25) (layer F.Fab) (width 0.1))
+    (fp_line (start -2.1 -1.7) (end -2.1 1.7) (layer F.CrtYd) (width 0.05))
+    (fp_line (start -2.1 1.7) (end 2.1 1.7) (layer F.CrtYd) (width 0.05))
+    (fp_line (start 2.1 1.7) (end 2.1 -1.7) (layer F.CrtYd) (width 0.05))
+    (fp_line (start 2.1 -1.7) (end -2.1 -1.7) (layer F.CrtYd) (width 0.05))
+    (pad 4 smd rect (at -1.1 -0.85 180) (size 1.4 1.2) (layers F.Cu F.Paste F.Mask)
+      (net 1 "Net-(C1-Pad2)"))
+    (pad 3 smd rect (at 1.1 -0.85 180) (size 1.4 1.2) (layers F.Cu F.Paste F.Mask)
+      (net 2 GND))
+    (pad 2 smd rect (at 1.1 0.85 180) (size 1.4 1.2) (layers F.Cu F.Paste F.Mask)
+      (net 3 "Net-(C2-Pad1)"))
+    (pad 1 smd rect (at -1.1 0.85 180) (size 1.4 1.2) (layers F.Cu F.Paste F.Mask)
+      (net 2 GND))
+    (model ${KISYS3DMOD}/Crystal.3dshapes/Crystal_SMD_3225-4Pin_3.2x2.5mm.wrl
+      (at (xyz 0 0 0))
+      (scale (xyz 1 1 1))
+      (rotate (xyz 0 0 0))
+    )
+  )
   (module random-keyboard-parts:SKQG-1155865 (layer F.Cu)
     (at 24.74475 37.0925)
@@
     (pad 1 smd rect (at 4.5 1.6) (size 2.25 0.5) (layers F.Cu F.Paste F.Mask)
       (net 2 GND))
-  )
-  (module Crystal:Crystal_SMD_3225-4Pin_3.2x2.5mm (layer F.Cu)
-    (at 43.67675 38.0755 180)
-    (descr "SMD Crystal SERIES SMD3225/4 http://www.txccrystal.com/images/pdf/7m-accuracy.pdf, 3.2x2.5mm^2 package")
-    (tags "SMD SMT crystal")
-    (attr smd)
-    (fp_text reference Y1 (at -0.01125 2.3885) (layer F.SilkS)
-      (effects (font (size 1 1) (thickness 0.15)))
-    )
-    (fp_text value Crystal_GND24_Small (at 0 2.45) (layer F.Fab)
-      (effects (font (size 1 1) (thickness 0.15)))
-    )
-    (fp_text user %R (at 0 0) (layer F.Fab)
-      (effects (font (size 0.7 0.7) (thickness 0.105)))
-    )
-    (fp_line (start -1.6 -1.25) (end -1.6 1.25) (layer F.Fab) (width 0.1))
-    (fp_line (start -1.6 1.25) (end 1.6 1.25) (layer F.Fab) (width 0.1))
-    (fp_line (start 1.6 1.25) (end 1.6 -1.25) (layer F.Fab) (width 0.1))
-    (fp_line (start 1.6 -1.25) (end -1.6 -1.25) (layer F.Fab) (width 0.1))
-    (fp_line (start -1.6 0.25) (end -0.6 1.25) (layer F.Fab) (width 0.1))
-    (fp_line (start -2 -1.65) (end -2 1.65) (layer F.SilkS) (width 0.12))
-    (fp_line (start -2 1.65) (end 2 1.65) (layer F.SilkS) (width 0.12))
-    (fp_line (start -2.1 -1.7) (end -2.1 1.7) (layer F.CrtYd) (width 0.05))
-    (fp_line (start -2.1 1.7) (end 2.1 1.7) (layer F.CrtYd) (width 0.05))
-    (fp_line (start 2.1 1.7) (end 2.1 -1.7) (layer F.CrtYd) (width 0.05))
-    (fp_line (start 2.1 -1.7) (end -2.1 -1.7) (layer F.CrtYd) (width 0.05))
-    (pad 4 smd rect (at -1.1 -0.85 180) (size 1.4 1.2) (layers F.Cu F.Paste F.Mask)
-      (net 1 "Net-(C1-Pad2)"))
-    (pad 3 smd rect (at 1.1 -0.85 180) (size 1.4 1.2) (layers F.Cu F.Paste F.Mask)
-      (net 2 GND))
-    (pad 2 smd rect (at 1.1 0.85 180) (size 1.4 1.2) (layers F.Cu F.Paste F.Mask)
-      (net 3 "Net-(C2-Pad1)"))
-    (pad 1 smd rect (at -1.1 0.85 180) (size 1.4 1.2) (layers F.Cu F.Paste F.Mask)
-      (net 2 GND))
-    (model ${KISYS3DMOD}/Crystal.3dshapes/Crystal_SMD_3225-4Pin_3.2x2.5mm.wrl
-      (at (xyz 0 0 0))
-      (scale (xyz 1 1 1))
-      (rotate (xyz 0 0 0))
-    )
   )
   (module Package_QFP:TQFP-44_10x10mm_P0.8mm (layer F.Cu)
@@
   (segment (start 27.84475 38.9425) (end 28.33575 38.9425) (width 0.381) (layer F.Cu) (net 2))
   (segment (start 28.33575 38.9425) (end 28.33575 38.0535) (width 0.381) (layer F.Cu) (net 2))
-  (segment (start 34.85224 36.48501) (end 35.96775 35.3695) (width 0.381) (layer F.Cu) (net 2))
+  (segment (start 34.925 36.48501) (end 36.04051 35.3695) (width 0.381) (layer F.Cu) (net 2))
   (segment (start 29.90424 36.48501) (end 34.85224 36.48501) (width 0.381) (layer F.Cu) (net 2))
   (segment (start 28.33575 38.0535) (end 29.90424 36.48501) (width 0.381) (layer F.Cu) (net 2))
@@
   (segment (start 47.72475 30.7335) (end 49.94275 32.9515) (width 0.381) (layer F.Cu) (net 2))
   (segment (start 46.11775 30.7335) (end 47.72475 30.7335) (width 0.381) (layer F.Cu) (net 2))
-  (segment (start 21.42275 30.8735) (end 21.42275 32.9235) (width 0.381) (layer F.Cu) (net 2))
-  (segment (start 21.42275 25.6235) (end 16.92275 25.6235) (width 0.381) (layer F.Cu) (net 2))
-  (segment (start 16.92275 25.6235) (end 16.92275 32.9235) (width 0.381) (layer F.Cu) (net 2))
-  (segment (start 16.92275 32.9235) (end 21.42275 32.9235) (width 0.381) (layer F.Cu) (net 2))
   (segment (start 39.85575 37.2255) (end 39.78275 37.1525) (width 0.254) (layer F.Cu) (net 3))
   (segment (start 42.57675 37.2255) (end 39.85575 37.2255) (width 0.254) (layer F.Cu) (net 3))
@@
   (segment (start 34.82975 32.7025) (end 32.67075 32.7025) (width 0.254) (layer B.Cu) (net 11))
   (segment (start 32.67075 32.7025) (end 30.76575 32.7025) (width 0.254) (layer F.Cu) (net 11))
-  (segment (start 24.18475 32.7025) (end 30.76575 32.7025) (width 0.254) (layer F.Cu) (net 11))
-  (segment (start 21.64475 35.2425) (end 24.18475 32.7025) (width 0.254) (layer F.Cu) (net 11))
+  (segment (start 25.4635 35.2425) (end 28.0035 32.7025) (width 0.254) (layer F.Cu) (net 11))
+  (segment (start 21.64475 35.2425) (end 25.4635 35.2425) (width 0.254) (layer F.Cu) (net 11))
+  (segment (start 28.0035 32.7025) (end 30.76575 32.7025) (width 0.254) (layer F.Cu) (net 11))
   (segment (start 24.79675 29.2735) (end 25.43175 29.9085) (width 0.254) (layer F.Cu) (net 12))
   (segment (start 21.42275 29.2735) (end 24.79675 29.2735) (width 0.254) (layer F.Cu) (net 12))
@@
   (segment (start 46.18175 22.6695) (end 46.11775 22.7335) (width 0.254) (layer F.Cu) (net 16))
   (segment (start 48.54575 22.6695) (end 46.18175 22.6695) (width 0.254) (layer F.Cu) (net 16))
+  (zone (net 2) (net_name GND) (layer F.Cu) (hatch edge 0.508)
+    (connect_pads yes (clearance 0.3))
+    (min_thickness 0.3)
+    (fill yes (arc_segments 32) (thermal_gap 0.508) (thermal_bridge_width 0.508) (smoothing fillet) (radius 2))
+    (polygon
+      (pts
+        (xy 49.657 40.386) (xy 37.973 40.386) (xy 37.846 34.29) (xy 49.657 34.29)
+      )
+    )
+  )
+  (zone (net 2) (net_name GND) (layer F.Cu) (hatch edge 0.508)
+    (connect_pads yes (clearance 0.3))
+    (min_thickness 0.3)
+    (fill yes (arc_segments 32) (thermal_gap 0.508) (thermal_bridge_width 0.508) (smoothing chamfer) (radius 1))
+    (polygon
+      (pts
+        (xy 45.72 32.004) (xy 35.179 32.004) (xy 35.179 21.463) (xy 45.72 21.463)
+      )
+    )
+  )
+  (zone (net 2) (net_name GND) (layer F.Cu) (hatch edge 0.508)
+    (connect_pads yes (clearance 0.2))
+    (min_thickness 0.2)
+    (fill yes (arc_segments 32) (thermal_gap 0.508) (thermal_bridge_width 0.508) (smoothing fillet) (radius 1))
+    (polygon
+      (pts
+        (xy 23.114 34.339812) (xy 15.367 34.339812) (xy 15.367 24.306812) (xy 23.114 24.306812)
+      )
+    )
+  )
 )
